Commit message: changed package name in files

File: urdf/links_joints.xacro (robot description, xacro)
@@ -51,5 +51,5 @@
                 <origin rpy="${leg_visualorigin_rpy}" xyz="0 0 0" />
                 <geometry>
-                    <mesh filename="package://robot_description/meshes/link_leftleg.STL" scale="0.001 0.001 0.001" />
+                    <mesh filename="package://autotuner/meshes/link_leftleg.STL" scale="0.001 0.001 0.001" />
                 </geometry>
                 <material name="Blue">
@@ -71,5 +71,5 @@
                 <origin rpy="${leg_visualorigin_rpy}" xyz="0 0 0" />
                 <geometry>
-                    <mesh filename="package://robot_description/meshes/link_rightleg.STL" scale="0.001 0.001 0.001" />
+                    <mesh filename="package://autotuner/meshes/link_rightleg.STL" scale="0.001 0.001 0.001" />
                 </geometry>
                 <material name="Blue">

File: urdf/robot.xacro (robot description, xacro)
@@ -2,5 +2,5 @@
 <robot name="ranch_rover" xmlns:xacro="https://ros.org/wiki/xacro">
     <!-- xacro files to be included-->
-    <xacro:include filename="$(find robot_description)/urdf/links_joints.xacro" />
+    <xacro:include filename="$(find autotuner)/urdf/links_joints.xacro" />
     <!-- First link of the robot. Corresponds to the robot main frame. -->
     <link name="link_chassis">
@@ -20,5 +20,5 @@
             <origin rpy="0 0 0" xyz="0 0 0" />
             <geometry>
-                <mesh filename="package://robot_description/meshes/link_chassis.STL" scale="0.001 0.001 0.001" />
+                <mesh filename="package://autotuner/meshes/link_chassis.STL" scale="0.001 0.001 0.001" />
             </geometry>
         </visual>
@@ -51,5 +51,5 @@
         <geometry>
             <mesh
-            filename="package://robot_description/meshes/base_link.STL" />
+            filename="package://autotuner/meshes/base_link.STL" />
         </geometry>
         <material
@@ -65,5 +65,5 @@
         <geometry>
             <mesh
-            filename="package://robot_description/meshes/base_link.STL" />
+            filename="package://autotuner/meshes/base_link.STL" />
         </geometry>
         </collision>
@@ -91,5 +91,5 @@
         <geometry>
             <mesh
-            filename="package://robot_description/meshes/Link_1.STL" />
+            filename="package://autotuner/meshes/Link_1.STL" />
         </geometry>
         <material
@@ -105,5 +105,5 @@
         <geometry>
             <mesh
-            filename="package://robot_description/meshes/Link_1.STL" />
+            filename="package://autotuner/meshes/Link_1.STL" />
         </geometry>
         </collision>
@@ -160,5 +160,5 @@
         <geometry>
             <mesh
-            filename="package://robot_description/meshes/Link_2.STL" />
+            filename="package://autotuner/meshes/Link_2.STL" />
         </geometry>
         <material
@@ -174,5 +174,5 @@
         <geometry>
             <mesh
-            filename="package://robot_description/meshes/Link_2.STL" />
+            filename="package://autotuner/meshes/Link_2.STL" />
         </geometry>
         </collision>
@@ -229,5 +229,5 @@
         <geometry>
             <mesh
-            filename="package://robot_description/meshes/Link_3.STL" />
+            filename="package://autotuner/meshes/Link_3.STL" />
         </geometry>
         <material
@@ -243,5 +243,5 @@
         <geometry>
             <mesh
-            filename="package://robot_description/meshes/Link_3.STL" />
+            filename="package://autotuner/meshes/Link_3.STL" />
         </geometry>
         </collision>
@@ -298,5 +298,5 @@
         <geometry>
             <mesh
-            filename="package://robot_description/meshes/Link_4.STL" />
+            filename="package://autotuner/meshes/Link_4.STL" />
         </geometry>
         <material
@@ -312,5 +312,5 @@
         <geometry>
             <mesh
-            filename="package://robot_description/meshes/Link_4.STL" />
+            filename="package://autotuner/meshes/Link_4.STL" />
         </geometry>
         </collision>

File: urdf/robot_original.xacro (robot description, xacro)
@@ -2,5 +2,5 @@
 <robot name="ranch_rover" xmlns:xacro="https://ros.org/wiki/xacro">
     <!-- xacro files to be included-->
-    <xacro:include filename="$(find robot_description)/urdf/links_joints.xacro" />
+    <xacro:include filename="$(find autotuner)/urdf/links_joints.xacro" />
     <!-- First link of the robot. Corresponds to the robot main frame. -->
     <link name="link_chassis">
@@ -20,5 +20,5 @@
             <origin rpy="0 0 0" xyz="0 0 0" />
             <geometry>
-                <mesh filename="package://robot_description/meshes/link_chassis.STL" scale="0.001 0.001 0.001" />
+                <mesh filename="package://autotuner/meshes/link_chassis.STL" scale="0.001 0.001 0.001" />
             </geometry>
         </visual>
@@ -51,5 +51,5 @@
         <geometry>
             <mesh
-            filename="package://robot_description/meshes/base_link.STL" />
+            filename="package://autotuner/meshes/base_link.STL" />
         </geometry>
         <material
@@ -65,5 +65,5 @@
         <geometry>
             <mesh
-            filename="package://robot_description/meshes/base_link.STL" />
+            filename="package://autotuner/meshes/base_link.STL" />
         </geometry>
         </collision>
@@ -91,5 +91,5 @@
         <geometry>
             <mesh
-            filename="package://robot_description/meshes/Link_1.STL" />
+            filename="package://autotuner/meshes/Link_1.STL" />
         </geometry>
         <material
@@ -105,5 +105,5 @@
         <geometry>
             <mesh
-            filename="package://robot_description/meshes/Link_1.STL" />
+            filename="package://autotuner/meshes/Link_1.STL" />
         </geometry>
         </collision>
@@ -160,5 +160,5 @@
         <geometry>
             <mesh
-            filename="package://robot_description/meshes/Link_2.STL" />
+            filename="package://autotuner/meshes/Link_2.STL" />
         </geometry>
         <material
@@ -174,5 +174,5 @@
         <geometry>
             <mesh
-            filename="package://robot_description/meshes/Link_2.STL" />
+            filename="package://autotuner/meshes/Link_2.STL" />
         </geometry>
         </collision>
@@ -229,5 +229,5 @@
         <geometry>
             <mesh
-            filename="package://robot_description/meshes/Link_3.STL" />
+            filename="package://autotuner/meshes/Link_3.STL" />
         </geometry>
         <material
@@ -243,5 +243,5 @@
         <geometry>
             <mesh
-            filename="package://robot_description/meshes/Link_3.STL" />
+            filename="package://autotuner/meshes/Link_3.STL" />
         </geometry>
         </collision>
@@ -298,5 +298,5 @@
         <geometry>
             <mesh
-            filename="package://robot_description/meshes/Link_4.STL" />
+            filename="package://autotuner/meshes/Link_4.STL" />
         </geometry>
         <material
@@ -312,5 +312,5 @@
         <geometry>
             <mesh
-            filename="package://robot_description/meshes/Link_4.STL" />
+            filename="package://autotuner/meshes/Link_4.STL" />
         </geometry>
         </collision>
