Commit message: started visualizer

File: urdf/robot_controlsim_v3_withSTL.urdf (robot description, URDF)
Before this commit: robot ranch_rover, 5 links, 4 joints
Links:
- link Link_1: geometry collision mesh filename=../meshes/Link_1.STL; visual mesh filename=../meshes/Link_1.STL
- link Link_2: geometry collision mesh filename=../meshes/Link_2.STL; visual mesh filename=../meshes/Link_2.STL
- link Link_3: geometry collision mesh filename=../meshes/Link_3.STL; visual mesh filename=../meshes/Link_3.STL
- link Link_4: geometry collision mesh filename=../meshes/Link_4.STL; visual mesh filename=../meshes/Link_4.STL
- link link_chassis: geometry collision mesh filename=../meshes/link_chassis.STL scale=0.001 0.001 0.001; visual mesh filename=../meshes/link_chassis.STL scale=0.001 0.001 0.001
